Commit message: using schunk_svh_description repo instead of svh driver

File: urdf/svh.urdf.xacro (robot description, xacro)
@@ -15,5 +15,5 @@
 	<origin xyz="0 0 -0.032" rpy="0 0 0" />
 	<geometry>
-          <mesh filename="package://schunk_svh_driver/description/meshes/base10.dae" />
+          <mesh filename="package://schunk_svh_description/meshes/base10.dae" />
 	</geometry>
       </visual>
@@ -21,5 +21,5 @@
 	<origin xyz="0 0 -0.032" rpy="0 0 0" />
 	<geometry>
-          <mesh filename="package://schunk_svh_driver/description/meshes/base10.dae" />
+          <mesh filename="package://schunk_svh_description/meshes/base10.dae" />
 	</geometry>
       </collision>
@@ -56,5 +56,5 @@
 	<origin rpy="0 0 0" xyz="0 0.01313 0" />
 	<geometry>
-          <mesh scale="${side*(1)} 1 1" filename="package://schunk_svh_driver/description/meshes/h10.dae" />
+          <mesh scale="${side*(1)} 1 1" filename="package://schunk_svh_description/meshes/h10.dae" />
 	</geometry>
       </visual>
@@ -62,5 +62,5 @@
 	<origin rpy="0 0 0" xyz="0 0.01313 0" />
 	<geometry>
-          <mesh scale="${side*(1)} 1 1" filename="package://schunk_svh_driver/description/meshes/h10.dae" />
+          <mesh scale="${side*(1)} 1 1" filename="package://schunk_svh_description/meshes/h10.dae" />
 	</geometry>
       </collision>
@@ -71,5 +71,5 @@
 	<origin xyz="${side*(-0.0007)} 0 -0.01002" />
 	<geometry>
-          <mesh scale="${side*(1)} 1 1" filename="package://schunk_svh_driver/description/meshes/h11.dae" />
+          <mesh scale="${side*(1)} 1 1" filename="package://schunk_svh_description/meshes/h11.dae" />
 	</geometry>
       </visual>
@@ -77,5 +77,5 @@
 	<origin xyz="${side*(-0.0007)} 0 -0.01002" />
 	<geometry>
-          <mesh scale="${side*(1)} 1 1" filename="package://schunk_svh_driver/description/meshes/h11.dae" />
+          <mesh scale="${side*(1)} 1 1" filename="package://schunk_svh_description/meshes/h11.dae" />
 	</geometry>
       </collision>
@@ -118,5 +118,5 @@
 	<origin xyz="0 0 0.02442" />
 	<geometry>
-          <mesh scale="1 ${side*(1)} 1" filename="package://schunk_svh_driver/description/meshes/d10.dae" />
+          <mesh scale="1 ${side*(1)} 1" filename="package://schunk_svh_description/meshes/d10.dae" />
 	</geometry>
       </visual>
@@ -124,5 +124,5 @@
 	<origin xyz="0 0 0.02442" />
 	<geometry>
-          <mesh scale="1 ${side*(1)} 1" filename="package://schunk_svh_driver/description/meshes/d10.dae" />
+          <mesh scale="1 ${side*(1)} 1" filename="package://schunk_svh_description/meshes/d10.dae" />
 	</geometry>
       </collision>
@@ -132,10 +132,10 @@
       <visual>
 	<geometry>
-          <mesh scale="1 ${side*(1)} ${side*(1)}" filename="package://schunk_svh_driver/description/meshes/d11.dae" />
-	</geometry>
-      </visual>
-      <collision>
-	<geometry>
-          <mesh scale="1 ${side*(1)} ${side*(1)}" filename="package://schunk_svh_driver/description/meshes/d11.dae" />
+          <mesh scale="1 ${side*(1)} ${side*(1)}" filename="package://schunk_svh_description/meshes/d11.dae" />
+	</geometry>
+      </visual>
+      <collision>
+	<geometry>
+          <mesh scale="1 ${side*(1)} ${side*(1)}" filename="package://schunk_svh_description/meshes/d11.dae" />
 	</geometry>
       </collision>
@@ -144,10 +144,10 @@
       <visual>
 	<geometry>
-          <mesh scale="1 ${side*(1)} ${side*(1)}" filename="package://schunk_svh_driver/description/meshes/d12.dae" />
-	</geometry>
-      </visual>
-      <collision>
-	<geometry>
-          <mesh scale="1 ${side*(1)} ${side*(1)}" filename="package://schunk_svh_driver/description/meshes/d12.dae" />
+          <mesh scale="1 ${side*(1)} ${side*(1)}" filename="package://schunk_svh_description/meshes/d12.dae" />
+	</geometry>
+      </visual>
+      <collision>
+	<geometry>
+          <mesh scale="1 ${side*(1)} ${side*(1)}" filename="package://schunk_svh_description/meshes/d12.dae" />
 	</geometry>
       </collision>
@@ -156,10 +156,10 @@
       <visual>
 	<geometry>
-          <mesh scale="1 ${side*(1)} ${side*(1)}" filename="package://schunk_svh_driver/description/meshes/d13.dae" />
-	</geometry>
-      </visual>
-      <collision>
-	<geometry>
-          <mesh scale="1 ${side*(1)} ${side*(1)}" filename="package://schunk_svh_driver/description/meshes/d13.dae" />
+          <mesh scale="1 ${side*(1)} ${side*(1)}" filename="package://schunk_svh_description/meshes/d13.dae" />
+	</geometry>
+      </visual>
+      <collision>
+	<geometry>
+          <mesh scale="1 ${side*(1)} ${side*(1)}" filename="package://schunk_svh_description/meshes/d13.dae" />
 	</geometry>
       </collision>
@@ -170,5 +170,5 @@
 	<origin xyz="0 0 0.01321" />
 	<geometry>
-          <mesh filename="package://schunk_svh_driver/description/meshes/f10.dae" />
+          <mesh filename="package://schunk_svh_description/meshes/f10.dae" />
 	</geometry>
       </visual>
@@ -176,5 +176,5 @@
 	<origin xyz="0 0 0.01321" />
 	<geometry>
-          <mesh filename="package://schunk_svh_driver/description/meshes/f10.dae" />
+          <mesh filename="package://schunk_svh_description/meshes/f10.dae" />
 	</geometry>
       </collision>
@@ -183,10 +183,10 @@
       <visual>
 	<geometry>
-          <mesh filename="package://schunk_svh_driver/description/meshes/f11.dae" />
-	</geometry>
-      </visual>
-      <collision>
-	<geometry>
-          <mesh filename="package://schunk_svh_driver/description/meshes/f11.dae" />
+          <mesh filename="package://schunk_svh_description/meshes/f11.dae" />
+	</geometry>
+      </visual>
+      <collision>
+	<geometry>
+          <mesh filename="package://schunk_svh_description/meshes/f11.dae" />
 	</geometry>
       </collision>
@@ -195,10 +195,10 @@
       <visual>
 	<geometry>
-          <mesh filename="package://schunk_svh_driver/description/meshes/f12.dae" />
-	</geometry>
-      </visual>
-      <collision>
-	<geometry>
-          <mesh filename="package://schunk_svh_driver/description/meshes/f12.dae" />
+          <mesh filename="package://schunk_svh_description/meshes/f12.dae" />
+	</geometry>
+      </visual>
+      <collision>
+	<geometry>
+          <mesh filename="package://schunk_svh_description/meshes/f12.dae" />
 	</geometry>
       </collision>
@@ -207,10 +207,10 @@
       <visual>
 	<geometry>
-          <mesh filename="package://schunk_svh_driver/description/meshes/f13.dae" />
-	</geometry>
-      </visual>
-      <collision>
-	<geometry>
-          <mesh filename="package://schunk_svh_driver/description/meshes/f13.dae" />
+          <mesh filename="package://schunk_svh_description/meshes/f13.dae" />
+	</geometry>
+      </visual>
+      <collision>
+	<geometry>
+          <mesh filename="package://schunk_svh_description/meshes/f13.dae" />
 	</geometry>
       </collision>
@@ -221,5 +221,5 @@
 	<origin xyz="0 0 0.01321" />
 	<geometry>
-          <mesh filename="package://schunk_svh_driver/description/meshes/f20.dae" />
+          <mesh filename="package://schunk_svh_description/meshes/f20.dae" />
 	</geometry>
       </visual>
@@ -227,5 +227,5 @@
 	<origin xyz="0 0 0.01321" />
 	<geometry>
-          <mesh filename="package://schunk_svh_driver/description/meshes/f20.dae" />
+          <mesh filename="package://schunk_svh_description/meshes/f20.dae" />
 	</geometry>
       </collision>
@@ -234,10 +234,10 @@
       <visual>
 	<geometry>
-          <mesh filename="package://schunk_svh_driver/description/meshes/f21.dae" />
-	</geometry>
-      </visual>
-      <collision>
-	<geometry>
-          <mesh filename="package://schunk_svh_driver/description/meshes/f21.dae" />
+          <mesh filename="package://schunk_svh_description/meshes/f21.dae" />
+	</geometry>
+      </visual>
+      <collision>
+	<geometry>
+          <mesh filename="package://schunk_svh_description/meshes/f21.dae" />
 	</geometry>
       </collision>
@@ -246,10 +246,10 @@
       <visual>
 	<geometry>
-          <mesh filename="package://schunk_svh_driver/description/meshes/f22.dae" />
-	</geometry>
-      </visual>
-      <collision>
-	<geometry>
-          <mesh filename="package://schunk_svh_driver/description/meshes/f22.dae" />
+          <mesh filename="package://schunk_svh_description/meshes/f22.dae" />
+	</geometry>
+      </visual>
+      <collision>
+	<geometry>
+          <mesh filename="package://schunk_svh_description/meshes/f22.dae" />
 	</geometry>
       </collision>
@@ -258,10 +258,10 @@
       <visual>
 	<geometry>
-          <mesh filename="package://schunk_svh_driver/description/meshes/f23.dae" />
-	</geometry>
-      </visual>
-      <collision>
-	<geometry>
-          <mesh filename="package://schunk_svh_driver/description/meshes/f23.dae" />
+          <mesh filename="package://schunk_svh_description/meshes/f23.dae" />
+	</geometry>
+      </visual>
+      <collision>
+	<geometry>
+          <mesh filename="package://schunk_svh_description/meshes/f23.dae" />
 	</geometry>
       </collision>
@@ -272,5 +272,5 @@
 	<origin xyz="0 0 -0.01321" />
 	<geometry>
-          <mesh filename="package://schunk_svh_driver/description/meshes/f30.dae" />
+          <mesh filename="package://schunk_svh_description/meshes/f30.dae" />
 	</geometry>
       </visual>
@@ -278,5 +278,5 @@
 	<origin xyz="0 0 -0.01321" />
 	<geometry>
-          <mesh filename="package://schunk_svh_driver/description/meshes/f30.dae" />
+          <mesh filename="package://schunk_svh_description/meshes/f30.dae" />
 	</geometry>
       </collision>
@@ -285,10 +285,10 @@
       <visual>
 	<geometry>
-          <mesh filename="package://schunk_svh_driver/description/meshes/f31.dae" />
-	</geometry>
-      </visual>
-      <collision>
-	<geometry>
-          <mesh filename="package://schunk_svh_driver/description/meshes/f31.dae" />
+          <mesh filename="package://schunk_svh_description/meshes/f31.dae" />
+	</geometry>
+      </visual>
+      <collision>
+	<geometry>
+          <mesh filename="package://schunk_svh_description/meshes/f31.dae" />
 	</geometry>
       </collision>
@@ -297,10 +297,10 @@
       <visual>
 	<geometry>
-          <mesh filename="package://schunk_svh_driver/description/meshes/f32.dae" />
-	</geometry>
-      </visual>
-      <collision>
-	<geometry>
-          <mesh filename="package://schunk_svh_driver/description/meshes/f32.dae" />
+          <mesh filename="package://schunk_svh_description/meshes/f32.dae" />
+	</geometry>
+      </visual>
+      <collision>
+	<geometry>
+          <mesh filename="package://schunk_svh_description/meshes/f32.dae" />
 	</geometry>
       </collision>
@@ -309,10 +309,10 @@
       <visual>
 	<geometry>
-          <mesh filename="package://schunk_svh_driver/description/meshes/f33.dae" />
-	</geometry>
-      </visual>
-      <collision>
-	<geometry>
-          <mesh filename="package://schunk_svh_driver/description/meshes/f33.dae" />
+          <mesh filename="package://schunk_svh_description/meshes/f33.dae" />
+	</geometry>
+      </visual>
+      <collision>
+	<geometry>
+          <mesh filename="package://schunk_svh_description/meshes/f33.dae" />
 	</geometry>
       </collision>
@@ -323,5 +323,5 @@
 	<origin xyz="0 0 -0.01321" />
 	<geometry>
-          <mesh filename="package://schunk_svh_driver/description/meshes/f40.dae" />
+          <mesh filename="package://schunk_svh_description/meshes/f40.dae" />
 	</geometry>
       </visual>
@@ -329,5 +329,5 @@
 	<origin xyz="0 0 -0.01321" />
 	<geometry>
-          <mesh filename="package://schunk_svh_driver/description/meshes/f40.dae" />
+          <mesh filename="package://schunk_svh_description/meshes/f40.dae" />
 	</geometry>
       </collision>
@@ -336,10 +336,10 @@
       <visual>
 	<geometry>
-          <mesh filename="package://schunk_svh_driver/description/meshes/f41.dae" />
-	</geometry>
-      </visual>
-      <collision>
-	<geometry>
-          <mesh filename="package://schunk_svh_driver/description/meshes/f41.dae" />
+          <mesh filename="package://schunk_svh_description/meshes/f41.dae" />
+	</geometry>
+      </visual>
+      <collision>
+	<geometry>
+          <mesh filename="package://schunk_svh_description/meshes/f41.dae" />
 	</geometry>
       </collision>
@@ -348,10 +348,10 @@
       <visual>
 	<geometry>
-          <mesh filename="package://schunk_svh_driver/description/meshes/f42.dae" />
-	</geometry>
-      </visual>
-      <collision>
-	<geometry>
-          <mesh filename="package://schunk_svh_driver/description/meshes/f42.dae" />
+          <mesh filename="package://schunk_svh_description/meshes/f42.dae" />
+	</geometry>
+      </visual>
+      <collision>
+	<geometry>
+          <mesh filename="package://schunk_svh_description/meshes/f42.dae" />
 	</geometry>
       </collision>
@@ -360,10 +360,10 @@
       <visual>
 	<geometry>
-          <mesh filename="package://schunk_svh_driver/description/meshes/f43.dae" />
-	</geometry>
-      </visual>
-      <collision>
-	<geometry>
-          <mesh filename="package://schunk_svh_driver/description/meshes/f43.dae" />
+          <mesh filename="package://schunk_svh_description/meshes/f43.dae" />
+	</geometry>
+      </visual>
+      <collision>
+	<geometry>
+          <mesh filename="package://schunk_svh_description/meshes/f43.dae" />
 	</geometry>
       </collision>
