Commit message: Gazebo sim effort control

File: urdf/svh.urdf.xacro (robot description, xacro)
@@ -1,6 +1,9 @@
 <?xml version="1.0"?>
 <robot xmlns:xacro="http://www.ros.org/wiki/xacro">
+  <xacro:include filename="$(find schunk_svh_description)/urdf/common.xacro" />
+  <xacro:include filename="$(find schunk_svh_description)/urdf/svh.transmission.xacro" />
+  <xacro:include filename="$(find schunk_svh_description)/urdf/svh.gazebo.xacro" />
   <xacro:property name="cyl_radius" value="0.001" />
-  <xacro:macro name="svh" params="parent name side *origin">
+  <xacro:macro name="svh" params="parent name side *origin robot_namespace:='/'">
     <!-- RIGHT HAND = 1, LEFT HAND = -1 -->
     <!-- BASE_LINE LINKS -->
@@ -13,15 +16,20 @@
       <xacro:insert_block name="origin" />
       <visual>
-	<origin xyz="0 0 -0.032" rpy="0 0 0" />
-	<geometry>
+        <xacro:insert_block name="origin" />
+        <geometry>
           <mesh filename="package://schunk_svh_description/meshes/base10.dae" />
 	</geometry>
       </visual>
       <collision>
-	<origin xyz="0 0 -0.032" rpy="0 0 0" />
-	<geometry>
+        <xacro:insert_block name="origin" />
+        <geometry>
           <mesh filename="package://schunk_svh_description/meshes/base10.dae" />
 	</geometry>
       </collision>
+      <inertial>
+        <mass value="0.57743"/>
+        <origin xyz="0.0 -2.3e-05 0.139371"/>
+        <inertia ixx="0.04725" ixy="-0.0" ixz="-0.0" iyy="0.04717" iyz="0.0" izz="0.07606" />
+      </inertial>
     </link>
     <link name="${name}_d">
@@ -32,4 +40,5 @@
       <!-- 	<material name="${name}_green" /> -->
       <!-- </visual> -->
+      <xacro:default_inertial mass="0.01"/>
     </link>
     <link name="${name}_h">
@@ -41,4 +50,5 @@
       <!-- 	<material name="${name}_green" /> -->
       <!-- </visual> -->
+      <xacro:default_inertial mass="0.01"/>
     </link>
     <link name="${name}_d2">
@@ -50,4 +60,5 @@
       <!-- 	<material name="${name}_green" /> -->
       <!-- </visual> -->
+      <xacro:default_inertial mass="0.01"/>
     </link>
     <!-- LENGTH NOT FOUND IN DATASHEET! GUESSED!!! -->
@@ -65,4 +76,5 @@
 	</geometry>
       </collision>
+      <xacro:default_inertial mass="0.01"/>
     </link>
     <!-- LENGTH NOT FOUND IN DATASHEET! GUESSED!!! -->
@@ -80,4 +92,9 @@
 	</geometry>
       </collision>
+      <inertial>
+        <mass value="0.46184"/>
+        <origin xyz="0.145071 -0.037868 0.323449"/>
+        <inertia ixx="0.01908" ixy="-0.00121" ixz="-0.00011" iyy="0.01704" iyz="0.00277" izz="0.00862"/>
+      </inertial>
     </link>
     <!-- LENGTH NOT FOUND IN DATASHEET! GUESSED!!! -->
@@ -90,4 +107,5 @@
       <!-- 	<material name="green" /> -->
       <!-- </visual> -->
+      <xacro:default_inertial mass="0.01"/>
     </link>
     <link name="${name}_e">
@@ -102,4 +120,5 @@
       <!-- 	<material name="green" /> -->
       <!-- </visual> -->
+      <xacro:default_inertial mass="0.01"/>
     </link>
     <!-- LENGTH NOT FOUND IN DATASHEET! GUESSED, BUT POSITION CALCULATED: E5 = D-G!!! -->
@@ -112,4 +131,5 @@
       <!-- 	<material name="green" /> -->
       <!-- </visual> -->
+      <xacro:default_inertial mass="0.01"/>
     </link>
     <!-- THUMB LINKS -->
@@ -127,6 +147,13 @@
 	</geometry>
       </collision>
-    </link>
-    <link name="${name}_virtual_a" />
+      <inertial>
+        <mass value="0.0739"/>
+        <origin xyz="0.0 0.002024 0.178636"/>
+        <inertia ixx="0.00103" ixy="-0.0" ixz="-0.0" iyy="0.00165" iyz="4e-05" izz="0.00111"/>
+      </inertial>
+    </link>
+    <link name="${name}_virtual_a">
+      <xacro:default_inertial mass="0.01"/>
+    </link>
     <link name="${name}_a">
       <visual>
@@ -140,4 +167,9 @@
 	</geometry>
       </collision>
+      <inertial>
+        <mass value="0.41222"/>
+        <origin xyz="0.240205 0.010733 0.00019"/>
+        <inertia ixx="0.00413" ixy="0.00073" ixz="-0.0" iyy="0.01679" iyz="0.0" izz="0.01796"/>
+      </inertial>
     </link>
     <link name="${name}_b">
@@ -152,4 +184,9 @@
 	</geometry>
       </collision>
+      <inertial>
+        <mass value="0.08224"/>
+        <origin xyz="0.123157 -0.008382 -2.7e-05"/>
+        <inertia ixx="0.00089" ixy="5e-05" ixz="0.0" iyy="0.00139" iyz="0.0" izz="0.00103"/>
+      </inertial>
     </link>
     <link name="${name}_c">
@@ -164,4 +201,9 @@
 	</geometry>
       </collision>
+      <inertial>
+        <mass value="0.06198"/>
+        <origin xyz="0.113729 0.01094 0.0"/>
+        <inertia ixx="0.00025" ixy="-0.0" ixz="-0.0" iyy="0.00051" iyz="0.0" izz="0.00052"/>
+      </inertial>
     </link>
     <!-- INDEX FINGER LINKS -->
@@ -179,4 +221,9 @@
 	</geometry>
       </collision>
+      <inertial>
+        <mass value="0.02383"/>
+        <origin xyz="0.003634 0.000206 -0.09885"/>
+        <inertia ixx="0.00021" ixy="-0.0" ixz="-1e-05" iyy="0.00011" iyz="-0.0" izz="0.00019"/>
+      </inertial>
     </link>
     <link name="${name}_l">
@@ -191,4 +238,9 @@
 	</geometry>
       </collision>
+      <inertial>
+        <mass value="0.13003"/>
+        <origin xyz="0.261673 0.003521 0.0"/>
+        <inertia ixx="0.00051" ixy="-3e-05" ixz="0.0" iyy="0.00335" iyz="-0.0" izz="0.00344"/>
+      </inertial>
     </link>
     <link name="${name}_p">
@@ -203,4 +255,9 @@
 	</geometry>
       </collision>
+      <inertial>
+        <mass value="0.03264"/>
+        <origin xyz="0.1384 -0.004609 0.0"/>
+        <inertia ixx="0.00016" ixy="-0.0" ixz="0.0" iyy="0.00031" iyz="-0.0" izz="0.00024"/>
+      </inertial>
     </link>
     <link name="${name}_t">
@@ -215,4 +272,9 @@
 	</geometry>
       </collision>
+      <inertial>
+        <mass value="0.0324"/>
+        <origin xyz="0.102924 0.000592 0.0"/>
+        <inertia ixx="9e-05" ixy="-1e-05" ixz="-0.0" iyy="0.00017" iyz="0.0" izz="0.00017"/>
+      </inertial>
     </link>
     <!-- MIDDLE FINGER LINKS -->
@@ -230,4 +292,9 @@
 	</geometry>
       </collision>
+      <inertial>
+        <mass value="0.02377"/>
+        <origin xyz="0.003357 -8e-06 -0.099643"/>
+        <inertia ixx="0.00021" ixy="-0.0" ixz="-1e-05" iyy="0.00011" iyz="0.0" izz="0.00019"/>
+      </inertial>
     </link>
     <link name="${name}_k">
@@ -242,4 +309,9 @@
 	</geometry>
       </collision>
+      <inertial>
+        <mass value="0.13474"/>
+        <origin xyz="0.271122 0.00413 0.0"/>
+        <inertia ixx="0.00052" ixy="-3e-05" ixz="-0.0" iyy="0.0037" iyz="-0.0" izz="0.0038"/>
+      </inertial>
     </link>
     <link name="${name}_o">
@@ -254,4 +326,9 @@
 	</geometry>
       </collision>
+      <inertial>
+        <mass value="0.0422"/>
+        <origin xyz="0.16683 -0.003774 0.0"/>
+        <inertia ixx="0.0002" ixy="0.0" ixz="-0.0" iyy="0.00047" iyz="0.0" izz="0.0004"/>
+      </inertial>
     </link>
     <link name="${name}_s">
@@ -266,4 +343,9 @@
 	</geometry>
       </collision>
+      <inertial>
+        <mass value="0.03239"/>
+        <origin xyz="0.102794 0.00042 0.0"/>
+        <inertia ixx="9e-05" ixy="-1e-05" ixz="0.0" iyy="0.00017" iyz="0.0" izz="0.00017"/>
+      </inertial>
     </link>
     <!-- RING FINGER LINKS -->
@@ -281,4 +363,9 @@
 	</geometry>
       </collision>
+      <inertial>
+        <mass value="0.02377"/>
+        <origin xyz="0.003805 0.000386 0.100079"/>
+        <inertia ixx="0.00021" ixy="0.0" ixz="1e-05" iyy="0.00011" iyz="-0.0" izz="0.00019"/>
+      </inertial>
     </link>
     <link name="${name}_j">
@@ -293,4 +380,9 @@
 	</geometry>
       </collision>
+      <inertial>
+        <mass value="0.1377"/>
+        <origin xyz="0.258283 -0.00154 0.0"/>
+        <inertia ixx="0.00055" ixy="0.00018" ixz="-0.0" iyy="0.00411" iyz="0.0" izz="0.00426"/>
+      </inertial>
     </link>
     <link name="${name}_n">
@@ -305,4 +397,9 @@
 	</geometry>
       </collision>
+      <inertial>
+        <mass value="0.04207"/>
+        <origin xyz="0.166851 -0.00362 0.0"/>
+        <inertia ixx="0.00019" ixy="0.0" ixz="-0.0" iyy="0.00047" iyz="0.0" izz="0.0004"/>
+      </inertial>
     </link>
     <link name="${name}_r">
@@ -317,4 +414,9 @@
 	</geometry>
       </collision>
+      <inertial>
+        <mass value="0.03229"/>
+        <origin xyz="0.102676 0.000301 0.0"/>
+        <inertia ixx="9e-05" ixy="-1e-05" ixz="0.0" iyy="0.00017" iyz="-0.0" izz="0.00017"/>
+      </inertial>
     </link>
     <!-- LITTLE FINGER LINKS -->
@@ -332,4 +434,9 @@
 	</geometry>
       </collision>
+      <inertial>
+        <mass value="0.02377"/>
+        <origin xyz="0.003653 4.4e-05 0.100085"/>
+        <inertia ixx="0.00021" ixy="0.0" ixz="1e-05" iyy="0.00011" iyz="-0.0" izz="0.00019"/>
+      </inertial>
     </link>
     <link name="${name}_i">
@@ -344,4 +451,9 @@
 	</geometry>
       </collision>
+      <inertial>
+        <mass value="0.12544"/>
+        <origin xyz="0.232293 0.00622 0.0"/>
+        <inertia ixx="0.00049" ixy="6e-05" ixz="-0.0" iyy="0.00316" iyz="0.0" izz="0.00328"/>
+      </inertial>
     </link>
     <link name="${name}_m">
@@ -356,4 +468,9 @@
 	</geometry>
       </collision>
+      <inertial>
+        <mass value="0.02488"/>
+        <origin xyz="0.119665 -0.009328 0.0"/>
+        <inertia ixx="0.00013" ixy="-0.0" ixz="-0.0" iyy="0.00023" iyz="0.0" izz="0.00016"/>
+      </inertial>
     </link>
     <link name="${name}_q">
@@ -368,4 +485,9 @@
 	</geometry>
       </collision>
+      <inertial>
+        <mass value="0.03234"/>
+        <origin xyz="0.102896 0.000307 0.0"/>
+        <inertia ixx="9e-05" ixy="-1e-05" ixz="-0.0" iyy="0.00017" iyz="0.0" izz="0.00017"/>
+      </inertial>
     </link>
     <joint name="${name}_Thumb_Flexion" type="revolute">
@@ -410,11 +532,12 @@
       <origin xyz="0 -0.01313 0" rpy="0 0 0" />
     </joint>
-    <joint name="${name}_j5" type="revolute">
-      <parent link="${name}_e1" />
-      <child link="${name}_e2" />
-      <limit effort="1000.0" lower="0.0" upper="0.98786" velocity="1" />
+    <!-- J5 JOINTS is set to fixed temporarily due to defective DH algo -->
+    <joint name="${name}_j5" type="fixed">
+      <parent link="${name}_e1"/>
+      <child link="${name}_e2"/>
+      <!--limit effort="1000.0" lower="0.0" upper="0.98786" velocity="1"/-->
       <origin xyz="${side*(0.01840)} 0.006 0.0375" rpy="0 0 0" />
-      <axis xyz="0 0 ${side*(1)}" />
-      <mimic joint="${name}_Thumb_Opposition" multiplier="1" offset="0" />
+      <!--axis xyz="0 0 ${side*(1)}"/-->
+      <!--mimic joint="${name}_Thumb_Opposition" multiplier="1" offset="0"/-->
     </joint>
     <joint name="${name}_f5" type="fixed">
@@ -578,4 +701,6 @@
       <axis xyz="0 0 ${side*(1)}" />
     </joint>
+    <xacro:svh_transmission name="${name}" />
+    <xacro:svh_gazebo name="${name}" robot_namespace="${robot_namespace}" />
 </xacro:macro>
 </robot>
