Commit message: Pass SVH parameters via the xacro file
This is currently hard-coded for firmware 2.3.

File: urdf/schunk_svh_driver.xacro (robot description, xacro)
@@ -7,5 +7,5 @@
         </xacro:svh>
         <!-- Individual joint configuration -->
-        <xacro:macro name="joint_ros2_control" params="name">
+        <xacro:macro name="joint_ros2_control" params="name **config">
                 <joint name="${name}">
                         <command_interface name="position">
@@ -16,17 +16,72 @@
                         <state_interface name="velocity"/>
                         <state_interface name="current"/>
+                        <xacro:insert_block name="config" />
                 </joint>
         </xacro:macro>
         <!-- ROS2 control interfaces -->
         <ros2_control name="schunk_svh_driver" type="system">
-                <xacro:joint_ros2_control name="Right_Hand_Thumb_Opposition"/>
-                <xacro:joint_ros2_control name="Right_Hand_Thumb_Flexion"/>
-                <xacro:joint_ros2_control name="Right_Hand_Index_Finger_Proximal"/>
-                <xacro:joint_ros2_control name="Right_Hand_Index_Finger_Distal"/>
-                <xacro:joint_ros2_control name="Right_Hand_Middle_Finger_Proximal"/>
-                <xacro:joint_ros2_control name="Right_Hand_Middle_Finger_Distal"/>
-                <xacro:joint_ros2_control name="Right_Hand_Finger_Spread"/>
-                <xacro:joint_ros2_control name="Right_Hand_Pinky"/>
-                <xacro:joint_ros2_control name="Right_Hand_Ring_Finger"/>
+                <xacro:joint_ros2_control name="Right_Hand_Thumb_Opposition">
+                        <config>
+                                <param name="position_controller">-1.0e+6, 1.0e+6,  50.0e+3, 1.00, 1.0e-3, -2000.0, 2000.0, 0.6, 0.1, 2000.0</param>
+                                <param name="current_controller">-605.0, 605.0, 0.405, 10.0e-6, -0.125 , 0.125, 0, 1984, -248.0, 248.0</param>
+                                <param name="home_settings">+1, -135.0e+3,  -5.0e+3, -15.0e+3, 0.99, 0.75</param>
+                        </config>
+                </xacro:joint_ros2_control>
+                <xacro:joint_ros2_control name="Right_Hand_Thumb_Flexion">
+                        <config>
+                                <param name="position_controller">-1.0e+6, 1.0e+6,  65.0e+3, 1.00, 1.0e-3, -2000.0, 2000.0, 0.6, 0.1, 2000.0</param>
+                                <param name="current_controller">-605.0, 605.0, 0.405, 10.0e-6, -0.125, 0.125, 0.0 , 1984, -248.0, 248.0</param>
+                                <param name="home_settings">+1, -105.0e+3,  -5.0e+3, -15.0e+3, 0.97, 0.75</param>
+                        </config>
+                </xacro:joint_ros2_control>
+                <xacro:joint_ros2_control name="Right_Hand_Index_Finger_Proximal">
+                        <config>
+                                <param name="position_controller">-1.0e+6, 1.0e+6,  40.0e+3, 1.00, 1.0e-3, -2000.0, 2000.0, 0.2, 0.17, 1600</param>
+                                <param name="current_controller">-350.0, 350.0, 0.405, 10.0e-6, -0.125 , 0.125 , 0, 1984, -248.0, 248.0</param>
+                                <param name="home_settings">-1,  2.0e+3,  42.0e+3,   -8.0e+3, 0.8, 0.75</param>
+                        </config>
+                </xacro:joint_ros2_control>
+                <xacro:joint_ros2_control name="Right_Hand_Index_Finger_Distal">
+                        <config>
+                                <param name="position_controller">-1.0e+6, 1.0e+6,  25.0e+3, 1.00, 1.0e-3, -1000.0, 1000.0, 0.4, 0.36, 2400</param>
+                                <param name="current_controller">-360.0, 360.0, 0.405, 10.0e-6, -0.125, 0.125, 0, 1984, -248.0, 248.0</param>
+                                <param name="home_settings">+1,  -47.0e+3,  -2.0e+3,  -8.0e+3, 1.33, 0.75</param>
+                        </config>
+                </xacro:joint_ros2_control>
+                <xacro:joint_ros2_control name="Right_Hand_Middle_Finger_Proximal">
+                        <config>
+                                <param name="position_controller">-1.0e+6, 1.0e+6,  40.0e+3, 1.00, 1.0e-3, -2000.0, 2000.0, 0.2, 0.17, 1600</param>
+                                <param name="current_controller">-350.0, 350.0, 0.405, 10.0e-6, -0.125 , 0.125 , 0, 1984, -248.0, 248.0</param>
+                                <param name="home_settings">-1,  2.0e+3,  42.0e+3,   -8.0e+3, 0.8, 0.75</param>
+                        </config>
+                </xacro:joint_ros2_control>
+                <xacro:joint_ros2_control name="Right_Hand_Middle_Finger_Distal">
+                        <config>
+                                <param name="position_controller">-1.0e+6, 1.0e+6,  25.0e+3, 1.00, 1.0e-3, -1000.0, 1000.0, 0.4, 0.36, 2400</param>
+                                <param name="current_controller">-360.0, 360.0, 0.405, 10.0e-6, -0.125, 0.125, 0, 1984, -248.0, 248.0</param>
+                                <param name="home_settings">+1,  -47.0e+3,  -2.0e+3,  -8.0e+3, 1.33, 0.75</param>
+                        </config>
+                </xacro:joint_ros2_control>
+                <xacro:joint_ros2_control name="Right_Hand_Finger_Spread">
+                        <config>
+                                <param name="position_controller">-1.0e+6, 1.0e+6,  25.0e+3, 1.00, 1.0e-3, -1000.0, 1000.0, 1.0, 0.36, 4000</param>
+                                <param name="current_controller">-500.0, 500.0, 0.405, 10.0e-6, -0.125 , 0.125 , 0, 1984, -248.0, 248.0</param>
+                                <param name="home_settings">+1,  -52.0e+3,  -2.0e+3,  -25.0e+3,0.58, 0.4</param>
+                        </config>
+                </xacro:joint_ros2_control>
+                <xacro:joint_ros2_control name="Right_Hand_Pinky">
+                        <config>
+                                <param name="position_controller">-1.0e+6, 1.0e+6,  20.0e+3, 1.00, 1.0e-3, -1000.0, 1000.0, 0.6, 0.0, 2500</param>
+                                <param name="current_controller">-360.0, 360.0, 0.405, 10.0e-6, -0.125, 0.125, 0, 1984, -248.0, 248.0</param>
+                                <param name="home_settings">+1,  -47.0e+3,  -2.0e+3,  -8.0e+3, 0.98, 0.75</param>
+                        </config>
+                </xacro:joint_ros2_control>
+                <xacro:joint_ros2_control name="Right_Hand_Ring_Finger">
+                        <config>
+                                <param name="position_controller">-1.0e+6, 1.0e+6,  20.0e+3, 1.00, 1.0e-3, -1000.0, 1000.0, 0.6, 0.0, 2500</param>
+                                <param name="current_controller">-360.0, 360.0, 0.405, 10.0e-6, -0.125, 0.125, 0, 1984, -248.0, 248.0</param>
+                                <param name="home_settings">+1,  -47.0e+3,  -2.0e+3,  -8.0e+3, 0.98, 0.75</param>
+                        </config>
+                </xacro:joint_ros2_control>
                 <hardware>
                         <plugin>schunk_svh_driver/SystemInterface</plugin>

Commit message: Use default parameters for unrecognized hand versions
We now use default parameters if the detected SVH version is not
directly supported. Supported versions have explicit parameter entries
in the xacro definition.

File: urdf/schunk_svh_driver.xacro (robot description, xacro)
@@ -4,5 +4,5 @@
         <link name="base_link" />
         <xacro:svh parent="base_link" name="Right_Hand" side="1"> <!-- left hand side=-1 -->
-                <origin xyz="0 0 0"  rpy= "0 0 0" />
+                <origin xyz="0 0 0"  rpy="0 0 0" />
         </xacro:svh>
         <!-- Individual joint configuration -->
@@ -28,67 +28,95 @@
                 Pinky
                 Finger_Spread
+        The system interface checks the SVH's firmware and loads the corresponding parameters.
         -->
         <ros2_control name="schunk_svh_driver" type="system">
                 <xacro:joint_ros2_control name="Right_Hand_Thumb_Flexion">
                         <config>
-                                <param name="position_controller">-1.0e+6 1.0e+6 65.0e+3 1.00 1.0e-3 -2000.0 2000.0 0.6 0.1 2000.0</param>
-                                <param name="current_controller">-605.0 605.0 0.405 10.0e-6 -0.125 0.125 0.0 1984 -248.0 248.0</param>
-                                <param name="home_settings">+1 -105.0e+3 -5.0e+3 -15.0e+3 0.97 0.75</param>
+                                <param name="2.3.position_controller">-1.0e+6 1.0e+6 65.0e+3 1.00 1.0e-3 -2000.0 2000.0 0.6 0.1 2000.0</param>
+                                <param name="2.3.current_controller">-605.0 605.0 0.405 10.0e-6 -0.125 0.125 0.0 1984 -248.0 248.0</param>
+                                <param name="2.3.home_settings">+1 -105.0e+3 -5.0e+3 -15.0e+3 0.97 0.75</param>
+                                <param name="0.0.position_controller">-1.0e+6 1.0e+6 65.0e+3 1.00 1.0e-3 -500.0 500.0 0.5 0.0 400.0</param>
+                                <param name="0.0.current_controller">-500.0 500.0 0.405 4.0e-6 -25.0 25.0 0.6 10 -255.0 255.0</param>
+                                <param name="0.0.home_settings">+1 -175.0e+3 -5.0e+3 -15.0e+3 0.97 0.75</param>
                         </config>
                 </xacro:joint_ros2_control>
                 <xacro:joint_ros2_control name="Right_Hand_Thumb_Opposition">
                         <config>
-                                <param name="position_controller">-1.0e+6 1.0e+6 50.0e+3 1.00 1.0e-3 -2000.0 2000.0 0.6 0.1 2000.0</param>
-                                <param name="current_controller">-605.0 605.0 0.405 10.0e-6 -0.125 0.125 0 1984 -248.0 248.0</param>
-                                <param name="home_settings">+1 -135.0e+3 -5.0e+3 -15.0e+3 0.99 0.75</param>
+                                <param name="2.3.position_controller">-1.0e+6 1.0e+6 50.0e+3 1.00 1.0e-3 -2000.0 2000.0 0.6 0.1 2000.0</param>
+                                <param name="2.3.current_controller">-605.0 605.0 0.405 10.0e-6 -0.125 0.125 0 1984 -248.0 248.0</param>
+                                <param name="2.3.home_settings">+1 -135.0e+3 -5.0e+3 -15.0e+3 0.99 0.75</param>
+                                <param name="0.0.position_controller">-1.0e+6 1.0e+6 50.0e+3 1.00 1.0e-3 -500.0 500.0 0.5 0.0 100.0</param>
+                                <param name="0.0.current_controller">-500.0 500.0 0.405 4.0e-6 -25.0 25.0 0.6 10 -255.0 255.0</param>
+                                <param name="0.0.home_settings">+1 -105.0e+3 -5.0e+3 -15.0e+3 0.99 0.75</param>
                         </config>
                 </xacro:joint_ros2_control>
                 <xacro:joint_ros2_control name="Right_Hand_Index_Finger_Distal">
                         <config>
-                                <param name="position_controller">-1.0e+6 1.0e+6 25.0e+3 1.00 1.0e-3 -1000.0 1000.0 0.4 0.36 2400</param>
-                                <param name="current_controller">-360.0 360.0 0.405 10.0e-6 -0.125 0.125 0 1984 -248.0 248.0</param>
-                                <param name="home_settings">+1 -47.0e+3 -2.0e+3 -8.0e+3 1.33 0.75</param>
+                                <param name="2.3.position_controller">-1.0e+6 1.0e+6 25.0e+3 1.00 1.0e-3 -1000.0 1000.0 0.4 0.36 2400</param>
+                                <param name="2.3.current_controller">-360.0 360.0 0.405 10.0e-6 -0.125 0.125 0 1984 -248.0 248.0</param>
+                                <param name="2.3.home_settings">+1 -47.0e+3 -2.0e+3 -8.0e+3 1.33 0.75</param>
+                                <param name="0.0.position_controller">-1.0e+6 1.0e+6 45.0e+3 1.00 1.0e-3 -500.0 500.0 0.5 0.0 40.0</param>
+                                <param name="0.0.current_controller">-300.0 300.0 0.405 4.0e-6 -25.0 25.0 1 10.0 -255.0 255.0</param>
+                                <param name="0.0.home_settings">+1 -47.0e+3 -2.0e+3 -8.0e+3 1.33 0.75</param>
                         </config>
                 </xacro:joint_ros2_control>
                 <xacro:joint_ros2_control name="Right_Hand_Index_Finger_Proximal">
                         <config>
-                                <param name="position_controller">-1.0e+6 1.0e+6 40.0e+3 1.00 1.0e-3 -2000.0 2000.0 0.2 0.17 1600</param>
-                                <param name="current_controller">-350.0 350.0 0.405 10.0e-6 -0.125 0.125 0 1984 -248.0 248.0</param>
-                                <param name="home_settings">-1 2.0e+3 42.0e+3 -8.0e+3 0.8 0.75</param>
+                                <param name="2.3.position_controller">-1.0e+6 1.0e+6 40.0e+3 1.00 1.0e-3 -2000.0 2000.0 0.2 0.17 1600</param>
+                                <param name="2.3.current_controller">-350.0 350.0 0.405 10.0e-6 -0.125 0.125 0 1984 -248.0 248.0</param>
+                                <param name="2.3.home_settings">-1 2.0e+3 42.0e+3 -8.0e+3 0.8 0.75</param>
+                                <param name="0.0.position_controller">-1.0e+6 1.0e+6 40.0e+3 1.00 1.0e-3 -500.0 500.0 0.8 0.0 1000.0</param>
+                                <param name="0.0.current_controller">-350.0 350.0 0.405 4.0e-6 -25.0 25.0 1 10.0 -255.0 255.0</param>
+                                <param name="0.0.home_settings">-1 2.0e+3 42.0e+3 -8.0e+3 0.8 0.75</param>
                         </config>
                 </xacro:joint_ros2_control>
                 <xacro:joint_ros2_control name="Right_Hand_Middle_Finger_Distal">
                         <config>
-                                <param name="position_controller">-1.0e+6 1.0e+6 25.0e+3 1.00 1.0e-3 -1000.0 1000.0 0.4 0.36 2400</param>
-                                <param name="current_controller">-360.0 360.0 0.405 10.0e-6 -0.125 0.125 0 1984 -248.0 248.0</param>
-                                <param name="home_settings">+1 -47.0e+3 -2.0e+3 -8.0e+3 1.33 0.75</param>
+                                <param name="2.3.position_controller">-1.0e+6 1.0e+6 25.0e+3 1.00 1.0e-3 -1000.0 1000.0 0.4 0.36 2400</param>
+                                <param name="2.3.current_controller">-360.0 360.0 0.405 10.0e-6 -0.125 0.125 0 1984 -248.0 248.0</param>
+                                <param name="2.3.home_settings">+1 -47.0e+3 -2.0e+3 -8.0e+3 1.33 0.75</param>
+                                <param name="0.0.position_controller">-1.0e+6 1.0e+6 45.0e+3 1.00 1.0e-3 -500.0 500.0 0.5 0.0 10.0</param>
+                                <param name="0.0.current_controller">-300.0 300.0 0.405 4.0e-6 -25.0 25.0 1 10.0 -255.0 255.0</param>
+                                <param name="0.0.home_settings">+1 -47.0e+3 -2.0e+3 -8.0e+3 1.33 0.75</param>
                         </config>
                 </xacro:joint_ros2_control>
                 <xacro:joint_ros2_control name="Right_Hand_Middle_Finger_Proximal">
                         <config>
-                                <param name="position_controller">-1.0e+6 1.0e+6 40.0e+3 1.00 1.0e-3 -2000.0 2000.0 0.2 0.17 1600</param>
-                                <param name="current_controller">-350.0 350.0 0.405 10.0e-6 -0.125 0.125 0 1984 -248.0 248.0</param>
-                                <param name="home_settings">-1 2.0e+3 42.0e+3 -8.0e+3 0.8 0.75</param>
+                                <param name="2.3.position_controller">-1.0e+6 1.0e+6 40.0e+3 1.00 1.0e-3 -2000.0 2000.0 0.2 0.17 1600</param>
+                                <param name="2.3.current_controller">-350.0 350.0 0.405 10.0e-6 -0.125 0.125 0 1984 -248.0 248.0</param>
+                                <param name="2.3.home_settings">-1 2.0e+3 42.0e+3 -8.0e+3 0.8 0.75</param>
+                                <param name="0.0.position_controller">-1.0e+6 1.0e+6 40.0e+3 1.00 1.0e-3 -500.0 500.0 0.8 0.0 1000.0</param>
+                                <param name="0.0.current_controller">-350.0 350.0 0.405 4.0e-6 -25.0 25.0 1 10.0 -255.0 255.0</param>
+                                <param name="0.0.home_settings">-1 2.0e+3 42.0e+3 -8.0e+3 0.8 0.75</param>
                         </config>
                 </xacro:joint_ros2_control>
                 <xacro:joint_ros2_control name="Right_Hand_Ring_Finger">
                         <config>
-                                <param name="position_controller">-1.0e+6 1.0e+6 20.0e+3 1.00 1.0e-3 -1000.0 1000.0 0.6 0.0 2500</param>
-                                <param name="current_controller">-360.0 360.0 0.405 10.0e-6 -0.125 0.125 0 1984 -248.0 248.0</param>
-                                <param name="home_settings">+1 -47.0e+3 -2.0e+3 -8.0e+3 0.98 0.75</param>
+                                <param name="2.3.position_controller">-1.0e+6 1.0e+6 20.0e+3 1.00 1.0e-3 -1000.0 1000.0 0.6 0.0 2500</param>
+                                <param name="2.3.current_controller">-360.0 360.0 0.405 10.0e-6 -0.125 0.125 0 1984 -248.0 248.0</param>
+                                <param name="2.3.home_settings">+1 -47.0e+3 -2.0e+3 -8.0e+3 0.98 0.75</param>
+                                <param name="0.0.position_controller">-1.0e+6 1.0e+6 45.0e+3 1.00 1.0e-3 -500.0 500.0 0.5 0.0 100.0</param>
+                                <param name="0.0.current_controller">-300.0 300.0 0.405 4.0e-6 -10 10 1 25.0 -255.0 255.0</param>
+                                <param name="0.0.home_settings">+1 -47.0e+3 -2.0e+3 -8.0e+3 0.98 0.75</param>
                         </config>
                 </xacro:joint_ros2_control>
                 <xacro:joint_ros2_control name="Right_Hand_Pinky">
                         <config>
-                                <param name="position_controller">-1.0e+6 1.0e+6 20.0e+3 1.00 1.0e-3 -1000.0 1000.0 0.6 0.0 2500</param>
-                                <param name="current_controller">-360.0 360.0 0.405 10.0e-6 -0.125 0.125 0 1984 -248.0 248.0</param>
-                                <param name="home_settings">+1 -47.0e+3 -2.0e+3 -8.0e+3 0.98 0.75</param>
+                                <param name="2.3.position_controller">-1.0e+6 1.0e+6 20.0e+3 1.00 1.0e-3 -1000.0 1000.0 0.6 0.0 2500</param>
+                                <param name="2.3.current_controller">-360.0 360.0 0.405 10.0e-6 -0.125 0.125 0 1984 -248.0 248.0</param>
+                                <param name="2.3.home_settings">+1 -47.0e+3 -2.0e+3 -8.0e+3 0.98 0.75</param>
+                                <param name="0.0.position_controller">-1.0e+6 1.0e+6 45.0e+3 1.00 1.0e-3 -500.0 500.0 0.5 0.0 100.0</param>
+                                <param name="0.0.current_controller">-300.0 300.0 0.405 4.0e-6 -10 10 1 25 -255.0 255.0</param>
+                                <param name="0.0.home_settings">+1 -47.0e+3 -2.0e+3 -8.0e+3 0.98 0.75</param>
                         </config>
                 </xacro:joint_ros2_control>
                 <xacro:joint_ros2_control name="Right_Hand_Finger_Spread">
                         <config>
-                                <param name="position_controller">-1.0e+6 1.0e+6 25.0e+3 1.00 1.0e-3 -1000.0 1000.0 1.0 0.36 4000</param>
-                                <param name="current_controller">-500.0 500.0 0.405 10.0e-6 -0.125 0.125 0 1984 -248.0 248.0</param>
-                                <param name="home_settings">+1 -52.0e+3 -2.0e+3 -25.0e+3 0.58 0.4</param>
+                                <param name="2.3.position_controller">-1.0e+6 1.0e+6 25.0e+3 1.00 1.0e-3 -1000.0 1000.0 1.0 0.36 4000</param>
+                                <param name="2.3.current_controller">-500.0 500.0 0.405 10.0e-6 -0.125 0.125 0 1984 -248.0 248.0</param>
+                                <param name="2.3.home_settings">+1 -52.0e+3 -2.0e+3 -25.0e+3 0.58 0.4</param>
+                                <param name="0.0.position_controller">-1.0e+6 1.0e+6 25.0e+3 1.00 1.0e-3 -500.0 500.0 0.5 0.0 100.0</param>
+                                <param name="0.0.current_controller">-500.0 500.0 0.405 4.0e-6 -4.0 4.0 0.70 60.0 -255.0 255.0</param>
+                                <param name="0.0.home_settings">+1 -57.0e+3 -2.0e+3 -25.0e+3 0.58 0.4</param>
                         </config>
                 </xacro:joint_ros2_control>
