Commit message: Distinguish between `left` and `right` hand
Users can now specify whether they have a `left` or `right` Schunk SVH
via the `handedness` parameter on startup.

File: urdf/schunk_svh_driver.xacro (robot description, xacro)
@@ -3,7 +3,18 @@
         <xacro:include filename="$(find schunk_svh_description)/urdf/svh.urdf.xacro" />
         <link name="base_link" />
-        <xacro:svh parent="base_link" name="Right_Hand" side="1"> <!-- left hand side=-1 -->
-                <origin xyz="0 0 0"  rpy="0 0 0" />
-        </xacro:svh>
+        <!-- Use a launch file parameter to choose between right and left hand -->
+        <xacro:property name="handedness" value="$(arg handedness)"/>
+        <xacro:if value="${handedness == 'right'}">
+                <xacro:property name="Hand" value="Right_Hand" />
+                <xacro:svh parent="base_link" name="${Hand}" side="1">
+                        <origin xyz="0 0 0"  rpy="0 0 0" />
+                </xacro:svh>
+        </xacro:if>
+        <xacro:unless value="${handedness == 'right'}">
+                <xacro:property name="Hand" value="Left_Hand" />
+                <xacro:svh parent="base_link" name="${Hand}" side="-1">
+                        <origin xyz="0 0 0"  rpy="0 0 0" />
+                </xacro:svh>
+        </xacro:unless>
         <!-- Individual joint configuration -->
         <xacro:macro name="joint_ros2_control" params="name **config">
@@ -31,29 +42,29 @@
         -->
         <ros2_control name="schunk_svh_driver" type="system">
-                <xacro:joint_ros2_control name="Right_Hand_Thumb_Flexion">
+                <xacro:joint_ros2_control name="${Hand}_Thumb_Flexion">
                         <xacro:include filename="$(find schunk_svh_driver)/urdf/parameters/thumb_flexion.xacro"/>
                 </xacro:joint_ros2_control>
-                <xacro:joint_ros2_control name="Right_Hand_Thumb_Opposition">
+                <xacro:joint_ros2_control name="${Hand}_Thumb_Opposition">
                         <xacro:include filename="$(find schunk_svh_driver)/urdf/parameters/thumb_opposition.xacro"/>
                 </xacro:joint_ros2_control>
-                <xacro:joint_ros2_control name="Right_Hand_Index_Finger_Distal">
+                <xacro:joint_ros2_control name="${Hand}_Index_Finger_Distal">
                         <xacro:include filename="$(find schunk_svh_driver)/urdf/parameters/index_finger_distal.xacro"/>
                 </xacro:joint_ros2_control>
-                <xacro:joint_ros2_control name="Right_Hand_Index_Finger_Proximal">
+                <xacro:joint_ros2_control name="${Hand}_Index_Finger_Proximal">
                         <xacro:include filename="$(find schunk_svh_driver)/urdf/parameters/index_finger_proximal.xacro"/>
                 </xacro:joint_ros2_control>
-                <xacro:joint_ros2_control name="Right_Hand_Middle_Finger_Distal">
+                <xacro:joint_ros2_control name="${Hand}_Middle_Finger_Distal">
                         <xacro:include filename="$(find schunk_svh_driver)/urdf/parameters/middle_finger_distal.xacro"/>
                 </xacro:joint_ros2_control>
-                <xacro:joint_ros2_control name="Right_Hand_Middle_Finger_Proximal">
+                <xacro:joint_ros2_control name="${Hand}_Middle_Finger_Proximal">
                         <xacro:include filename="$(find schunk_svh_driver)/urdf/parameters/middle_finger_proximal.xacro"/>
                 </xacro:joint_ros2_control>
-                <xacro:joint_ros2_control name="Right_Hand_Ring_Finger">
+                <xacro:joint_ros2_control name="${Hand}_Ring_Finger">
                         <xacro:include filename="$(find schunk_svh_driver)/urdf/parameters/ring_finger.xacro"/>
                 </xacro:joint_ros2_control>
-                <xacro:joint_ros2_control name="Right_Hand_Pinky">
+                <xacro:joint_ros2_control name="${Hand}_Pinky">
                         <xacro:include filename="$(find schunk_svh_driver)/urdf/parameters/pinky.xacro"/>
                 </xacro:joint_ros2_control>
-                <xacro:joint_ros2_control name="Right_Hand_Finger_Spread">
+                <xacro:joint_ros2_control name="${Hand}_Finger_Spread">
                         <xacro:include filename="$(find schunk_svh_driver)/urdf/parameters/finger_spread.xacro"/>
                 </xacro:joint_ros2_control>

Commit message: Support left and right hand control on startup
We replace `handedness` with `control`.
That's a bit more intuitive and allows to use the launch parameter also
for the name of the respective joint trajectory controller.

File: urdf/schunk_svh_driver.xacro (robot description, xacro)
@@ -4,6 +4,6 @@
         <link name="base_link" />
         <!-- Use a launch file parameter to choose between right and left hand -->
-        <xacro:property name="handedness" value="$(arg handedness)"/>
-        <xacro:if value="${handedness == 'right'}">
+        <xacro:property name="control" value="$(arg control)"/>
+        <xacro:if value="${control == 'right_hand'}">
                 <xacro:property name="Hand" value="Right_Hand" />
                 <xacro:svh parent="base_link" name="${Hand}" side="1">
@@ -11,5 +11,5 @@
                 </xacro:svh>
         </xacro:if>
-        <xacro:unless value="${handedness == 'right'}">
+        <xacro:unless value="${control == 'right_hand'}">
                 <xacro:property name="Hand" value="Left_Hand" />
                 <xacro:svh parent="base_link" name="${Hand}" side="-1">
