Commit message: Add a minimal Gazebo example

File: schunk_svh_description/urdf/common.xacro (robot description, xacro)
@@ -48,13 +48,13 @@
       <type>transmission_interface/SimpleTransmission</type>
       <joint name="${jname}">
-      <hardwareInterface>hardware_interface/EffortJointInterface</hardwareInterface>
-<!--         <hardwareInterface>hardware_interface/PositionJointInterface</hardwareInterface> -->
-<!--         <hardwareInterface>hardware_interface/VelocityJointInterface</hardwareInterface> -->
+      <!-- <hardwareInterface>hardware_interface/EffortJointInterface</hardwareInterface> -->
+      <hardwareInterface>hardware_interface/PositionJointInterface</hardwareInterface>
+      <!-- <hardwareInterface>hardware_interface/VelocityJointInterface</hardwareInterface> -->
       </joint>
       <actuator name="${jname}_motor">
         <mechanicalReduction>1</mechanicalReduction>
-      <hardwareInterface>hardware_interface/EffortJointInterface</hardwareInterface>
-<!--         <hardwareInterface>hardware_interface/PositionJointInterface</hardwareInterface> -->
-<!--         <hardwareInterface>hardware_interface/VelocityJointInterface</hardwareInterface> -->
+        <!-- <hardwareInterface>hardware_interface/EffortJointInterface</hardwareInterface> -->
+        <hardwareInterface>hardware_interface/PositionJointInterface</hardwareInterface>
+        <!-- <hardwareInterface>hardware_interface/VelocityJointInterface</hardwareInterface> -->
       </actuator>
     </transmission>

File: schunk_svh_description/urdf/svh-standalone.urdf.xacro (robot description, xacro)
@@ -3,4 +3,10 @@
  <xacro:include filename="$(find schunk_svh_description)/urdf/svh.urdf.xacro" />
  <xacro:arg name="name_prefix" default="left_hand" />
+ <link name="world"/>
+ <joint name="world_joint" type="fixed">
+   <parent link="world"/>
+   <child link="base_link"/>
+   <origin rpy="0.0 0.0 0.0" xyz="0.0 0.0 0.0"/>
+ </joint>
  <link name="base_link" />
  <xacro:svh parent="base_link" name="$(arg name_prefix)" side="-1">

File: schunk_svh_description/urdf/svh.urdf.xacro (robot description, xacro)
@@ -1,4 +1,4 @@
 <?xml version="1.0"?>
-<robot xmlns:xacro="http://www.ros.org/wiki/xacro">
+<robot name="svh" xmlns:xacro="http://www.ros.org/wiki/xacro">
   <xacro:include filename="$(find schunk_svh_description)/urdf/common.xacro" />
   <xacro:include filename="$(find schunk_svh_description)/urdf/svh.transmission.xacro" />
@@ -703,4 +703,4 @@
     <xacro:svh_transmission name="${name}" />
     <xacro:svh_gazebo name="${name}" robot_namespace="${robot_namespace}" />
-</xacro:macro>
+  </xacro:macro>
 </robot>
