Commit message: Use MuJoCo's built-in position control for the joints
This is easier to understand and configure.
Also use an open-loop control with ROS2`s `joint_trajectory_controller` by
providing idealized position feedback.
This avoids oscillations and drifts.
We could also avoid those by having MuJoCo run orders of magnitude
faster than ROS2 control and using high-gain position servos.

File: schunk_svh_simulation/urdf/joint.urdf.xacro (robot description, xacro)
@@ -2,16 +2,7 @@
 <robot xmlns:xacro="http://www.ros.org/wiki/xacro">
         <!-- Individual joint. -->
-        <xacro:macro name="joint_interface" params="name p d">
+        <xacro:macro name="joint_interface" params="name">
                 <joint name="${name}">
-                        <command_interface name="position">
-                                <param name="min">-1</param>
-                                <param name="max">1</param>
-                        </command_interface>
-                        <command_interface name="velocity">
-                                <param name="min">-1</param>
-                                <param name="max">1</param>
-                        </command_interface>
-                        <param name="p">${p}</param>
-                        <param name="d">${d}</param>
+                        <command_interface name="position"/>
                         <state_interface name="position"/>
                         <state_interface name="velocity"/>

File: schunk_svh_simulation/urdf/robot.urdf.xacro (robot description, xacro)
@@ -8,10 +8,10 @@
         <!-- ROS2 control interfaces -->
         <ros2_control name="schunk_svh_simulation" type="system">
-                <xacro:joint_interface name="joint1" p="1000" d="0.5" />
-                <xacro:joint_interface name="joint2" p="1000" d="0.5" />
-                <xacro:joint_interface name="joint3" p="500" d="0.5" />
-                <xacro:joint_interface name="joint4" p="100" d="0.5" />
-                <xacro:joint_interface name="joint5" p="10" d="0.5" />
-                <xacro:joint_interface name="joint6" p="10" d="0.5" />
+                <xacro:joint_interface name="joint1"/>
+                <xacro:joint_interface name="joint2"/>
+                <xacro:joint_interface name="joint3"/>
+                <xacro:joint_interface name="joint4"/>
+                <xacro:joint_interface name="joint5"/>
+                <xacro:joint_interface name="joint6"/>
                 <hardware>
                         <plugin>schunk_svh_simulation/Simulator</plugin>
