Commit message: Correctly initialize the svh macro for simulation
I forgot that somehow in 0aea103

File: schunk_svh_simulation/urdf/schunk_svh_simulation.xacro (robot description, xacro)
@@ -3,4 +3,7 @@
         <xacro:include filename="$(find schunk_svh_description)/urdf/svh.urdf.xacro" />
         <link name="base_link" />
+        <xacro:svh parent="base_link" name="Right_Hand" side="1">
+                <origin xyz="0 0 0"  rpy="0 0 0" />
+        </xacro:svh>
         <!-- Individual joint configuration -->
         <xacro:macro name="joint_ros2_control" params="name">
